File: hw-rgb-lcd-rpi.kicad_pcb (KiCad board)
At the start: 2 copper layers, 65 x 30 mm, 15 parts, among them J1 lq043t1dg03, J2 minilaptop-lcd, P1 GPIO, P2 I2C, P3 BATT, P4 MINILAP SPARE, P5 P_LED, P6 BACKLIGHT, U1 RPi_A+_B+_2B_Hat

Commit message: Add a licence name to the silkscreen
Parts:
- moved REF*** 1.53 mm to (158.8, 115.1)
Other:
- board text added: "CERN-OHL"
Changed lines of the file:
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@@
-(kicad_pcb (version 4) (host pcbnew 4.0.4+dfsg1-stable)
+(kicad_pcb (version 4) (host pcbnew 4.0.2+dfsg1-2~bpo8+1-stable)
   (general
     (links 100)
     (no_connects 0)
-    (area 108.494999 89.408 189.955001 130.996)
+    (area 94.997001 80.97 189.955001 129.372)
     (thickness 1.6)
-    (drawings 10)
+    (drawings 11)
     (tracks 747)
     (zones 0)
@@
   )
   (module Symbols:OSHW-Logo_5.7x6mm_SilkScreen (layer F.Cu)
-    (at 158.623 116.586)
+    (at 158.75 115.062)
     (descr "Open Source Hardware Logo")
     (tags "Logo OSHW")
     (attr virtual)
-    (fp_text reference REF*** (at 0 0) (layer F.SilkS) hide
+    (fp_text reference REF*** (at 0 7.874) (layer F.SilkS) hide
       (effects (font (size 1 1) (thickness 0.15)))
     )
@@
       (xy 0.376964 -2.709982)) (layer F.SilkS) (width 0.01))
   )
+  (gr_text CERN-OHL (at 158.75 118.872) (layer F.SilkS)
+    (effects (font (size 0.8 0.8) (thickness 0.2)))
+  )
   (dimension 65.024 (width 0.3) (layer Dwgs.User)

Commit message: update design rules for via sizes after talking to hackvana
Other:
- net class Default: via_drill 0.4 -> 0.3
- net class Power: via_drill 0.4 -> 0.3
Changed lines of the file:
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@@
     (edge_width 0.15)
     (via_size 0.6)
-    (via_drill 0.4)
+    (via_drill 0.3)
     (via_min_size 0.6)
     (via_min_drill 0.3)
@@
     (trace_width 0.1524)
     (via_dia 0.6)
-    (via_drill 0.4)
+    (via_drill 0.3)
     (uvia_dia 0.3)
     (uvia_drill 0.1)
@@
     (trace_width 0.25)
     (via_dia 0.6)
-    (via_drill 0.4)
+    (via_drill 0.3)
     (uvia_dia 0.3)
     (uvia_drill 0.1)
